File: card/elec/layout/default/card.kicad_pcb (KiCad board)
At the start: 2 copper layers, 225.7 x 100.8 mm, 0 parts

Commit message: [NFC] antenna
Parts:
- added C1: 50V 50pF C0G ±5% 0402 Multilayer Ceramic Capacitors MLCC - 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, lib:C0402, F.Cu at (157.4, 106.0)
- added U1: , lib:HM-NFC-Class6-Antenna, F.Cu at (156.4, 106.8)
- added U2: , lib:XQFN-8_L1.6-W1.6-P0.50-BR, F.Cu at (155.3, 106.0)
Routing:
- net lb: track 0.00 -> 1.70 mm
- net la: track 0.00 -> 1.68 mm
Other:
- board size 225.7 x 100.8 mm -> 99 x 55 mm
- board text removed: "{{GITHASH}}"
