File: card/elec/layout/default/card.kicad_pcb (KiCad board)
At the start: 2 copper layers, 88.6 x 51 mm, 5 parts

Commit message: [DIODE] name
Other:
- board text added: "DIODE COMPUTERS, INC."
- board text removed: "DIODE INC. HW/SW"

Commit message: [OWAY] PCB
Other:
- board text added: "www.oway.io"
- board text removed: "DIODE COMPUTERS, INC."
